File: avbay.sch (KiCad schematic (older format))
At the start: 16 parts, among them P1 CONN_2, P2 CONN_6, P3 CONN_2, P4 CONN_2, P6 CONN_01X12, SW2 SW_PUSH, SW3 SW_PUSH

Commit message: Added pyro schematic
Parts:
- removed P1: CONN_2, symbol CONN_2
Connections:
- net OVERRIDE_RX renamed MCU/RADIO_RX
- net OVERRIDE_TX renamed MCU/RADIO_TX
Changed lines of the file:
@@
 $Descr A4 11693 8268
 encoding utf-8
-Sheet 1 3
+Sheet 1 4
 Title ""
-Date "20 oct 2014"
+Date "4 dec 2014"
 Rev ""
 Comp ""
@@
 F8 "RADIO_TX" I R 6900 4000 60
 F9 "RADIO_RX" I R 6900 4150 60
-F10 "VSSA" I L 4900 3550 60
-F11 "VDDA" I L 4900 3750 60
 F12 "LED0" I L 4900 4500 60
 F13 "LED1" I L 4900 4650 60
@@
 F24 "GPIO6" I R 6900 5200 60
 F25 "GPIO7" I R 6900 5300 60
+F26 "SENSE1" I L 4900 2700 60
+F27 "SENSE2" I L 4900 2800 60
+F28 "SENSE3" I L 4900 2900 60
+F29 "SENSE4" I L 4900 3000 60
+F30 "TRIGGER1" I L 4900 3100 60
+F31 "TRIGGER2" I L 4900 3200 60
+F32 "TRIGGER3" I L 4900 3300 60
+F33 "TRIGGER4" I L 4900 3400 60
 $EndSheet
 $Comp
@@
 $EndComp
 $Comp
-L CONN_2 P1
-U 1 1 5430FD2D
-P 3600 3650
-F 0 "P1" V 3550 3650 40  0000 C CNN
-F 1 "CONN_2" V 3650 3650 40  0000 C CNN
-F 2 "" H 3600 3650 60  0000 C CNN
-F 3 "" H 3600 3650 60  0000 C CNN
-	1    3600 3650
-	-1   0    0    1
-$EndComp
-$Comp
 L 3V3 #PWR01
 U 1 1 5430FF93
@@
 	1    0    0    -1
 $EndComp
-Text Label 8250 3950 0    60   ~ 0
-OVERRIDE_TX
-Text Label 8300 4300 0    60   ~ 0
-OVERRIDE_RX
 $Sheet
 S 950  5250 1850 1500
@@
 	8050 3700 6900 3700
 Wire Wire Line
-	6900 4000 8000 4000
-Wire Wire Line
-	8000 4000 8000 4650
-Wire Wire Line
-	8000 4650 8650 4650
-Wire Wire Line
-	8650 4650 8650 4500
-Wire Wire Line
-	6900 4150 7950 4150
-Wire Wire Line
-	7950 4150 7950 5050
-Wire Wire Line
-	7950 5050 8650 5050
-Wire Wire Line
-	8650 5050 8650 4900
-Wire Wire Line
-	8650 4900 8300 4900
-Wire Wire Line
-	8300 4900 8300 4150
-Wire Wire Line
-	8300 4150 8350 4150
-Wire Wire Line
-	8650 4500 8250 4500
-Wire Wire Line
-	8250 4500 8250 3950
+	6900 4000 8250 4000
+Wire Wire Line
+	6900 4150 8350 4150
 Wire Wire Line
 	8250 3950 8350 3950
-Wire Wire Line
-	4900 3550 3950 3550
-Wire Wire Line
-	3950 3750 4900 3750
 Wire Wire Line
 	7600 2700 7600 2650
@@
 Wire Wire Line
 	4050 6300 4200 6300
+$Sheet
+S 2500 1300 1800 1250
+U 5480E61F
+F0 "Pyro" 50
+F1 "Pyro.sch" 50
+F2 "SENSE1" I R 4300 1550 60
+F3 "TRIGGER1" I R 4300 2050 60
+F4 "SENSE2" I R 4300 1650 60
+F5 "TRIGGER2" I R 4300 2150 60
+F6 "SENSE3" I R 4300 1750 60
+F7 "TRIGGER3" I R 4300 2250 60
+F8 "SENSE4" I R 4300 1850 60
+F9 "TRIGGER4" I R 4300 2350 60
+$EndSheet
+Wire Wire Line
+	4300 1550 4850 1550
+Wire Wire Line
+	4850 1550 4850 2700
+Wire Wire Line
+	4850 2700 4900 2700
+Wire Wire Line
+	4900 2800 4800 2800
+Wire Wire Line
+	4800 2800 4800 1650
+Wire Wire Line
+	4800 1650 4300 1650
+Wire Wire Line
+	4300 1750 4750 1750
+Wire Wire Line
+	4750 1750 4750 2900
+Wire Wire Line
+	4750 2900 4900 2900
+Wire Wire Line
+	4900 3000 4700 3000
+Wire Wire Line
+	4700 3000 4700 1850
+Wire Wire Line
+	4700 1850 4300 1850
+Wire Wire Line
+	4300 2050 4650 2050
+Wire Wire Line
+	4650 2050 4650 3100
+Wire Wire Line
+	4650 3100 4900 3100
+Wire Wire Line
+	4900 3200 4600 3200
+Wire Wire Line
+	4600 3200 4600 2150
+Wire Wire Line
+	4600 2150 4300 2150
+Wire Wire Line
+	4300 2250 4550 2250
+Wire Wire Line
+	4550 2250 4550 3300
+Wire Wire Line
+	4550 3300 4900 3300
+Wire Wire Line
+	4900 3400 4500 3400
+Wire Wire Line
+	4500 3400 4500 2350
+Wire Wire Line
+	4500 2350 4300 2350
+Wire Wire Line
+	8250 4000 8250 3950
 $EndSCHEMATC

Commit message: Added pyro circuits
Parts:
- BT1: footprint ~ -> Pin_Headers:Pin_Header_Straight_1x02
- D1, D2, D3, D4: footprint (none) -> LEDs:LED-0805
- P1: renamed from P6; footprint (none) -> Pin_Headers:Pin_Header_Straight_1x12
- P2: footprint (none) -> Pin_Headers:Pin_Header_Angled_1x06
- P3, P4: footprint (none) -> Pin_Headers:Pin_Header_Straight_1x02
- R1: renamed from R2; footprint (none) -> Resistors_SMD:R_0805_HandSoldering
- R2: renamed from R3; footprint (none) -> Resistors_SMD:R_0805_HandSoldering
- R3: renamed from R4; footprint (none) -> Resistors_SMD:R_0805_HandSoldering
- R4: renamed from R5; footprint (none) -> Resistors_SMD:R_0805_HandSoldering
- renumbered SW2 to SW1, SW3 to SW2
Changed lines of the file:
@@
 LIBS:xbee
 LIBS:avbay-cache
-EELAYER 27 0
+EELAYER 25 0
 EELAYER END
 $Descr A4 11693 8268
@@
 F8 "RADIO_TX" I R 6900 4000 60
 F9 "RADIO_RX" I R 6900 4150 60
-F12 "LED0" I L 4900 4500 60
-F13 "LED1" I L 4900 4650 60
-F14 "LED2" I L 4900 4800 60
-F15 "LED3" I L 4900 4950 60
-F16 "BTN0" I L 4900 5200 60
-F17 "BTN1" I L 4900 5350 60
-F18 "GPIO0" I R 6900 4600 60
-F19 "GPIO1" I R 6900 4700 60
-F20 "GPIO2" I R 6900 4800 60
-F21 "GPIO3" I R 6900 4900 60
-F22 "GPIO4" I R 6900 5000 60
-F23 "GPIO5" I R 6900 5100 60
-F24 "GPIO6" I R 6900 5200 60
-F25 "GPIO7" I R 6900 5300 60
-F26 "SENSE1" I L 4900 2700 60
-F27 "SENSE2" I L 4900 2800 60
-F28 "SENSE3" I L 4900 2900 60
-F29 "SENSE4" I L 4900 3000 60
-F30 "TRIGGER1" I L 4900 3100 60
-F31 "TRIGGER2" I L 4900 3200 60
-F32 "TRIGGER3" I L 4900 3300 60
-F33 "TRIGGER4" I L 4900 3400 60
+F10 "LED0" I L 4900 4500 60
+F11 "LED1" I L 4900 4650 60
+F12 "LED2" I L 4900 4800 60
+F13 "LED3" I L 4900 4950 60
+F14 "BTN0" I L 4900 5200 60
+F15 "BTN1" I L 4900 5350 60
+F16 "GPIO0" I R 6900 4600 60
+F17 "GPIO1" I R 6900 4700 60
+F18 "GPIO2" I R 6900 4800 60
+F19 "GPIO3" I R 6900 4900 60
+F20 "GPIO4" I R 6900 5000 60
+F21 "GPIO5" I R 6900 5100 60
+F22 "GPIO6" I R 6900 5200 60
+F23 "GPIO7" I R 6900 5300 60
+F24 "SENSE1" I L 4900 2700 60
+F25 "SENSE2" I L 4900 2800 60
+F26 "SENSE3" I L 4900 2900 60
+F27 "SENSE4" I L 4900 3000 60
+F28 "TRIGGER1" I L 4900 3100 60
+F29 "TRIGGER2" I L 4900 3200 60
+F30 "TRIGGER3" I L 4900 3300 60
+F31 "TRIGGER4" I L 4900 3400 60
 $EndSheet
 $Comp
@@
 F 0 "P2" V 8350 2700 60  0000 C CNN
 F 1 "CONN_6" V 8450 2700 60  0000 C CNN
-F 2 "" H 8400 2700 60  0000 C CNN
+F 2 "Pin_Headers:Pin_Header_Angled_1x06" H 8400 2700 60  0001 C CNN
 F 3 "" H 8400 2700 60  0000 C CNN
 	1    8400 2700
@@
 F 0 "P3" V 8350 3600 40  0000 C CNN
 F 1 "CONN_2" V 8450 3600 40  0000 C CNN
-F 2 "" H 8400 3600 60  0000 C CNN
+F 2 "Pin_Headers:Pin_Header_Straight_1x02" H 8400 3600 60  0001 C CNN
 F 3 "" H 8400 3600 60  0000 C CNN
 	1    8400 3600
@@
 F 0 "P4" V 8650 4050 40  0000 C CNN
 F 1 "CONN_2" V 8750 4050 40  0000 C CNN
-F 2 "" H 8700 4050 60  0000 C CNN
+F 2 "Pin_Headers:Pin_Header_Straight_1x02" H 8700 4050 60  0001 C CNN
 F 3 "" H 8700 4050 60  0000 C CNN
 	1    8700 4050
@@
 $EndSheet
 $Comp
-L R R5
+L R R4
 U 1 1 5437A174
 P 4350 4500
-F 0 "R5" V 4430 4500 40  0000 C CNN
+F 0 "R4" V 4430 4500 40  0000 C CNN
 F 1 "48" V 4357 4501 40  0000 C CNN
-F 2 "" V 4280 4500 30  0000 C CNN
+F 2 "Resistors_SMD:R_0805_HandSoldering" V 4280 4500 30  0001 C CNN
 F 3 "" H 4350 4500 30  0000 C CNN
 	1    4350 4500
@@
 $EndComp
 $Comp
-L R R4
+L R R3
 U 1 1 5437A32D
 P 4100 4650
-F 0 "R4" V 4180 4650 40  0000 C CNN
+F 0 "R3" V 4180 4650 40  0000 C CNN
 F 1 "48" V 4107 4651 40  0000 C CNN
-F 2 "" V 4030 4650 30  0000 C CNN
+F 2 "Resistors_SMD:R_0805_HandSoldering" V 4030 4650 30  0001 C CNN
 F 3 "" H 4100 4650 30  0000 C CNN
 	1    4100 4650
@@
 $EndComp
 $Comp
-L R R3
+L R R2
 U 1 1 5437A376
 P 3850 4800
-F 0 "R3" V 3930 4800 40  0000 C CNN
+F 0 "R2" V 3930 4800 40  0000 C CNN
 F 1 "48" V 3857 4801 40  0000 C CNN
-F 2 "" V 3780 4800 30  0000 C CNN
+F 2 "Resistors_SMD:R_0805_HandSoldering" V 3780 4800 30  0001 C CNN
 F 3 "" H 3850 4800 30  0000 C CNN
 	1    3850 4800
@@
 $EndComp
 $Comp
-L R R2
+L R R1
 U 1 1 5437A3A4
 P 3600 4950
-F 0 "R2" V 3680 4950 40  0000 C CNN
+F 0 "R1" V 3680 4950 40  0000 C CNN
 F 1 "48" V 3607 4951 40  0000 C CNN
-F 2 "" V 3530 4950 30  0000 C CNN
+F 2 "Resistors_SMD:R_0805_HandSoldering" V 3530 4950 30  0001 C CNN
 F 3 "" H 3600 4950 30  0000 C CNN
 	1    3600 4950
@@
 F 0 "D4" H 3800 4600 50  0000 C CNN
 F 1 "LED" H 3800 4400 50  0000 C CNN
-F 2 "" H 3800 4500 60  0000 C CNN
+F 2 "LEDs:LED-0805" H 3800 4500 60  0001 C CNN
 F 3 "" H 3800 4500 60  0000 C CNN
 	1    3800 4500
@@
 F 0 "D3" H 3550 4750 50  0000 C CNN
 F 1 "LED" H 3550 4550 50  0000 C CNN
-F 2 "" H 3550 4650 60  0000 C CNN
+F 2 "LEDs:LED-0805" H 3550 4650 60  0001 C CNN
 F 3 "" H 3550 4650 60  0000 C CNN
 	1    3550 4650
@@
 F 0 "D2" H 3300 4900 50  0000 C CNN
 F 1 "LED" H 3300 4700 50  0000 C CNN
-F 2 "" H 3300 4800 60  0000 C CNN
+F 2 "LEDs:LED-0805" H 3300 4800 60  0001 C CNN
 F 3 "" H 3300 4800 60  0000 C CNN
 	1    3300 4800
@@
 F 0 "D1" H 3050 5050 50  0000 C CNN
 F 1 "LED" H 3050 4850 50  0000 C CNN
-F 2 "" H 3050 4950 60  0000 C CNN
+F 2 "LEDs:LED-0805" H 3050 4950 60  0001 C CNN
 F 3 "" H 3050 4950 60  0000 C CNN
 	1    3050 4950
@@
 $EndComp
 $Comp
-L SW_PUSH SW3
+L SW_PUSH SW2
 U 1 1 5437AA50
 P 4400 5200
-F 0 "SW3" H 4550 5310 50  0000 C CNN
+F 0 "SW2" H 4550 5310 50  0000 C CNN
 F 1 "SW_PUSH" H 4400 5120 50  0000 C CNN
-F 2 "" H 4400 5200 60  0000 C CNN
+F 2 "" H 4400 5200 60  0001 C CNN
 F 3 "" H 4400 5200 60  0000 C CNN
 	1    4400 5200
@@
 $EndComp
 $Comp
-L SW_PUSH SW2
+L SW_PUSH SW1
 U 1 1 5437AAF9
 P 3750 5350
-F 0 "SW2" H 3900 5460 50  0000 C CNN
+F 0 "SW1" H 3900 5460 50  0000 C CNN
 F 1 "SW_PUSH" H 3750 5270 50  0000 C CNN
-F 2 "" H 3750 5350 60  0000 C CNN
+F 2 "" H 3750 5350 60  0001 C CNN
 F 3 "" H 3750 5350 60  0000 C CNN
 	1    3750 5350
@@
 $EndComp
 $Comp
-L CONN_01X12 P6
+L CONN_01X12 P1
 U 1 1 5437E79B
 P 7750 6000
-F 0 "P6" H 7750 6650 50  0000 C CNN
+F 0 "P1" H 7750 6650 50  0000 C CNN
 F 1 "CONN_01X12" V 7850 6000 50  0000 C CNN
-F 2 "" H 7750 6000 60  0000 C CNN
+F 2 "Pin_Headers:Pin_Header_Straight_1x12" H 7750 6000 60  0001 C CNN
 F 3 "" H 7750 6000 60  0000 C CNN
 	1    7750 6000
@@
 F 0 "BT1" H 3750 6500 50  0000 C CNN
 F 1 "BATTERY" H 3750 6110 50  0000 C CNN
-F 2 "~" H 3750 6300 60  0000 C CNN
+F 2 "Pin_Headers:Pin_Header_Straight_1x02" H 3750 6300 60  0000 C CNN
 F 3 "~" H 3750 6300 60  0000 C CNN
 	1    3750 6300
