File: avbay.sch (KiCad schematic (older format))
At the start: 15 parts, among them P1 CONN_01X12, P2 CONN_6, P3 CONN_2, P4 CONN_2, SW1 SW_PUSH, SW2 SW_PUSH

Commit message: New MOSFETs
Parts:
- removed BT1: BATTERY, Pin_Headers:Pin_Header_Straight_1x02, symbol BATTERY
- removed P1: CONN_01X12, Pin_Headers:Pin_Header_Straight_1x12, symbol CONN_01X12
- removed P3, P4: CONN_2, Pin_Headers:Pin_Header_Straight_1x02, symbol CONN_2
- added P1, P4, P5: TERM_BLOCK_2.54MM_2POS, symbol TERM_BLOCK_2.54MM_2POS
- added P3: TERM_BLOCK_2.54MM_12POS, symbol TERM_BLOCK_2.54MM_12POS
Connections:
- net 3V3: now also P3.9 (P9)
- net GND: now also P1.2 (PM), P3.11 (P11), P3.12 (P12)
- net MCU/GPIO0: now also P3.1 (P1)
- net MCU/GPIO1: now also P3.2 (P2)
- net MCU/GPIO2: now also P3.3 (P3)
- net MCU/GPIO3: now also P3.4 (P4)
- net MCU/GPIO4: now also P3.5 (P5)
- net MCU/GPIO5: now also P3.6 (P6)
- net MCU/GPIO6: now also P3.7 (P7)
- net MCU/GPIO7: now also P3.8 (P8)
- net MCU/RADIO_RX: now also P5.2 (PM)
- net MCU/RADIO_TX: now also P5.1 (P1)
- net MCU/USART_RX: now also P4.2 (PM)
- net MCU/USART_TX: now also P4.1 (P1)
- net Sheet54375BB5/Vbatt: now also P1.1 (P1)
- new net +5V: P3.10 (P10)
Changed lines of the file:
@@
 LIBS:xbee
 LIBS:avbay-cache
-EELAYER 25 0
+EELAYER 27 0
 EELAYER END
 $Descr A4 11693 8268
@@
 Sheet 1 4
 Title ""
-Date "4 dec 2014"
+Date "6 dec 2014"
 Rev ""
 Comp ""
@@
 $EndComp
 $Comp
-L CONN_2 P3
-U 1 1 5430F3D3
-P 8400 3600
-F 0 "P3" V 8350 3600 40  0000 C CNN
-F 1 "CONN_2" V 8450 3600 40  0000 C CNN
-F 2 "Pin_Headers:Pin_Header_Straight_1x02" H 8400 3600 60  0001 C CNN
-F 3 "" H 8400 3600 60  0000 C CNN
-	1    8400 3600
-	1    0    0    -1
-$EndComp
-$Comp
-L CONN_2 P4
-U 1 1 5430F47A
-P 8700 4050
-F 0 "P4" V 8650 4050 40  0000 C CNN
-F 1 "CONN_2" V 8750 4050 40  0000 C CNN
-F 2 "Pin_Headers:Pin_Header_Straight_1x02" H 8700 4050 60  0001 C CNN
-F 3 "" H 8700 4050 60  0000 C CNN
-	1    8700 4050
-	1    0    0    -1
-$EndComp
-$Comp
-L 3V3 #PWR01
+L 3V3 #PWR5
 U 1 1 5430FF93
 P 7900 2400
-F 0 "#PWR01" H 7900 2500 40  0001 C CNN
+F 0 "#PWR5" H 7900 2500 40  0001 C CNN
 F 1 "3V3" H 7900 2525 40  0000 C CNN
 F 2 "" H 7900 2400 60  0000 C CNN
@@
 $EndComp
 $Comp
-L GND #PWR02
+L GND #PWR4
 U 1 1 5430FF99
 P 7600 2700
-F 0 "#PWR02" H 7600 2700 30  0001 C CNN
+F 0 "#PWR4" H 7600 2700 30  0001 C CNN
 F 1 "GND" H 7600 2630 30  0001 C CNN
 F 2 "" H 7600 2700 60  0000 C CNN
@@
 $EndComp
 $Comp
-L GND #PWR03
+L GND #PWR1
 U 1 1 5437A755
 P 2800 5050
-F 0 "#PWR03" H 2800 5050 30  0001 C CNN
+F 0 "#PWR1" H 2800 5050 30  0001 C CNN
 F 1 "GND" H 2800 4980 30  0001 C CNN
 F 2 "" H 2800 5050 60  0000 C CNN
@@
 $EndComp
 $Comp
-L GND #PWR04
+L GND #PWR3
 U 1 1 5437AD2F
 P 3350 5400
-F 0 "#PWR04" H 3350 5400 30  0001 C CNN
+F 0 "#PWR3" H 3350 5400 30  0001 C CNN
 F 1 "GND" H 3350 5330 30  0001 C CNN
 F 2 "" H 3350 5400 60  0000 C CNN
@@
 $EndComp
 $Comp
-L CONN_01X12 P1
-U 1 1 5437E79B
-P 7750 6000
-F 0 "P1" H 7750 6650 50  0000 C CNN
-F 1 "CONN_01X12" V 7850 6000 50  0000 C CNN
-F 2 "Pin_Headers:Pin_Header_Straight_1x12" H 7750 6000 60  0001 C CNN
-F 3 "" H 7750 6000 60  0000 C CNN
-	1    7750 6000
-	0    -1   1    0
-$EndComp
-$Comp
-L GND #PWR05
+L GND #PWR8
 U 1 1 5437EF10
 P 8700 5800
-F 0 "#PWR05" H 8700 5800 30  0001 C CNN
+F 0 "#PWR8" H 8700 5800 30  0001 C CNN
 F 1 "GND" H 8700 5730 30  0001 C CNN
 F 2 "" H 8700 5800 60  0000 C CNN
@@
 $EndComp
 $Comp
-L 3V3 #PWR06
+L 3V3 #PWR6
 U 1 1 5437EF24
-P 8000 5600
-F 0 "#PWR06" H 8000 5700 40  0001 C CNN
-F 1 "3V3" H 8000 5725 40  0000 C CNN
-F 2 "" H 8000 5600 60  0000 C CNN
-F 3 "" H 8000 5600 60  0000 C CNN
-	1    8000 5600
-	1    0    0    -1
-$EndComp
-$Comp
-L GND #PWR07
+P 8000 5700
+F 0 "#PWR6" H 8000 5800 40  0001 C CNN
+F 1 "3V3" H 8000 5825 40  0000 C CNN
+F 2 "" H 8000 5700 60  0000 C CNN
+F 3 "" H 8000 5700 60  0000 C CNN
+	1    8000 5700
+	1    0    0    -1
+$EndComp
+$Comp
+L GND #PWR2
 U 1 1 54449D6F
 P 3050 6700
-F 0 "#PWR07" H 3050 6700 30  0001 C CNN
+F 0 "#PWR2" H 3050 6700 30  0001 C CNN
 F 1 "GND" H 3050 6630 30  0001 C CNN
 F 2 "" H 3050 6700 60  0000 C CNN
@@
 	1    0    0    -1
 $EndComp
-$Comp
-L BATTERY BT1
-U 1 1 54449F40
-P 3750 6300
-F 0 "BT1" H 3750 6500 50  0000 C CNN
-F 1 "BATTERY" H 3750 6110 50  0000 C CNN
-F 2 "Pin_Headers:Pin_Header_Straight_1x02" H 3750 6300 60  0000 C CNN
-F 3 "~" H 3750 6300 60  0000 C CNN
-	1    3750 6300
-	1    0    0    -1
-$EndComp
 Wire Wire Line
 	7600 2650 8050 2650
@@
 	8700 5700 8700 5800
 Wire Wire Line
-	8000 5600 8000 5800
-Wire Wire Line
 	8100 5800 8100 5700
 Wire Wire Line
@@
 Connection ~ 8300 5700
 Wire Wire Line
-	8100 5700 8000 5700
-Connection ~ 8000 5700
-Wire Wire Line
-	2800 6300 3450 6300
+	2800 6300 3650 6300
 Wire Wire Line
 	4200 6550 3050 6550
@@
 	4200 6300 4200 6550
 Wire Wire Line
-	4050 6300 4200 6300
+	3850 6300 4200 6300
 $Sheet
 S 2500 1300 1800 1250
@@
 Wire Wire Line
 	8250 4000 8250 3950
+$Comp
+L +5V #PWR7
+U 1 1 54829384
+P 8100 5700
+F 0 "#PWR7" H 8100 5790 20  0001 C CNN
+F 1 "+5V" H 8100 5790 30  0000 C CNN
+F 2 "" H 8100 5700 60  0000 C CNN
+F 3 "" H 8100 5700 60  0000 C CNN
+	1    8100 5700
+	1    0    0    -1
+$EndComp
+Wire Wire Line
+	8000 5700 8000 5800
+$Comp
+L TERM_BLOCK_2.54MM_2POS P1
+U 1 1 5482A325
+P 3750 5800
+F 0 "P1" V 3700 5800 40  0000 C CNN
+F 1 "TERM_BLOCK_2.54MM_2POS" V 3800 5800 40  0000 C CNN
+F 2 "" H 3750 5800 60  0000 C CNN
+F 3 "" H 3750 5800 60  0000 C CNN
+	1    3750 5800
+	0    -1   -1   0
+$EndComp
+Wire Wire Line
+	3650 6300 3650 6150
+Wire Wire Line
+	3850 6150 3850 6300
+$Comp
+L TERM_BLOCK_2.54MM_12POS P3
+U 1 1 5482B57E
+P 7750 6150
+F 0 "P3" V 7700 6150 60  0000 C CNN
+F 1 "TERM_BLOCK_2.54MM_12POS" V 7800 6150 60  0000 C CNN
+F 2 "" H 7750 6150 60  0000 C CNN
+F 3 "" H 7750 6150 60  0000 C CNN
+	1    7750 6150
+	0    -1   1    0
+$EndComp
+$Comp
+L TERM_BLOCK_2.54MM_2POS P4
+U 1 1 5482BA94
+P 8400 3600
+F 0 "P4" V 8350 3600 40  0000 C CNN
+F 1 "TERM_BLOCK_2.54MM_2POS" V 8450 3600 40  0000 C CNN
+F 2 "" H 8400 3600 60  0000 C CNN
+F 3 "" H 8400 3600 60  0000 C CNN
+	1    8400 3600
+	1    0    0    -1
+$EndComp
+$Comp
+L TERM_BLOCK_2.54MM_2POS P5
+U 1 1 5482BF92
+P 8700 4050
+F 0 "P5" V 8650 4050 40  0000 C CNN
+F 1 "TERM_BLOCK_2.54MM_2POS" V 8750 4050 40  0000 C CNN
+F 2 "" H 8700 4050 60  0000 C CNN
+F 3 "" H 8700 4050 60  0000 C CNN
+	1    8700 4050
+	1    0    0    -1
+$EndComp
 $EndSCHEMATC
