File: Hardware/Pyro.sch (KiCad schematic (older format))
At the start: 10 parts, among them P6 TERM_BLOCK_2.54MM_2POS, P7 TERM_BLOCK_2.54MM_8POS, Q1 DMN2041LSD, Q2 BSS138DW, Q3 DMN2041LSD, Q4 BSS138DW

Commit message: Roughed out PCB layout
Known issues:
- SW_PUSH holes too small. New footprint needed
- Sensor footprints are completely wrong.
- Regulator footprints might not be correct.

Tasks:
- Place passives according to schematic (especially
  with decoupling capacitors.
- Condense layout as much as possible for
  smallest board size
- Route board
Parts:
- P6: footprint (none) -> Socket_Strips:Socket_Strip_Straight_1x02
- P7: footprint (none) -> Socket_Strips:Socket_Strip_Straight_1x08
- Q1, Q3: footprint (none) -> Housings_SOIC:SOIC-8_3.9x4.9mm_Pitch1.27mm
Changed lines of the file:
@@
 TRIGGER1
 $Comp
-L GND #PWR016
+L GND #PWR019
 U 1 1 54810205
 P 1400 3600
-F 0 "#PWR016" H 1400 3600 30  0001 C CNN
+F 0 "#PWR019" H 1400 3600 30  0001 C CNN
 F 1 "GND" H 1400 3530 30  0001 C CNN
 F 2 "" H 1400 3600 60  0000 C CNN
@@
 TRIGGER2
 $Comp
-L GND #PWR017
+L GND #PWR020
 U 1 1 54810E85
 P 4500 3000
-F 0 "#PWR017" H 4500 3000 30  0001 C CNN
+F 0 "#PWR020" H 4500 3000 30  0001 C CNN
 F 1 "GND" H 4500 2930 30  0001 C CNN
 F 2 "" H 4500 3000 60  0000 C CNN
@@
 F 0 "P6" V 900 3400 40  0000 C CNN
 F 1 "TERM_BLOCK_2.54MM_2POS" V 1000 3400 40  0000 C CNN
-F 2 "" H 950 3400 60  0000 C CNN
+F 2 "Socket_Strips:Socket_Strip_Straight_1x02" H 950 3400 60  0001 C CNN
 F 3 "" H 950 3400 60  0000 C CNN
 	1    950  3400
@@
 F 0 "P7" V 2950 3900 60  0000 C CNN
 F 1 "TERM_BLOCK_2.54MM_8POS" V 3050 3900 60  0000 C CNN
-F 2 "" H 3000 3900 60  0000 C CNN
+F 2 "Socket_Strips:Socket_Strip_Straight_1x08" H 3000 3900 60  0001 C CNN
 F 3 "" H 3000 3900 60  0000 C CNN
 	1    3000 3900
@@
 F 0 "Q1" H 1100 2301 40  0000 R CNN
 F 1 "DMN2041LSD" H 1100 2600 40  0000 R CNN
-F 2 "" H 970 2552 29  0000 C CNN
+F 2 "Housings_SOIC:SOIC-8_3.9x4.9mm_Pitch1.27mm" H 970 2552 29  0001 C CNN
 F 3 "" H 1100 2450 60  0000 C CNN
 	1    1100 2450
@@
 F 0 "Q3" H 5800 2301 40  0000 R CNN
 F 1 "DMN2041LSD" H 5800 2600 40  0000 R CNN
-F 2 "" H 5670 2552 29  0000 C CNN
+F 2 "Housings_SOIC:SOIC-8_3.9x4.9mm_Pitch1.27mm" H 5670 2552 29  0001 C CNN
 F 3 "" H 5800 2450 60  0000 C CNN
 	1    5800 2450
@@
 F 0 "Q1" H 3550 2301 40  0000 R CNN
 F 1 "DMN2041LSD" H 3550 2600 40  0000 R CNN
-F 2 "" H 3420 2552 29  0000 C CNN
+F 2 "Housings_SOIC:SOIC-8_3.9x4.9mm_Pitch1.27mm" H 3420 2552 29  0001 C CNN
 F 3 "" H 3550 2450 60  0000 C CNN
 	2    3550 2450
@@
 F 0 "Q3" H 8050 2301 40  0000 R CNN
 F 1 "DMN2041LSD" H 8050 2600 40  0000 R CNN
-F 2 "" H 7920 2552 29  0000 C CNN
+F 2 "Housings_SOIC:SOIC-8_3.9x4.9mm_Pitch1.27mm" H 7920 2552 29  0001 C CNN
 F 3 "" H 8050 2450 60  0000 C CNN
 	2    8050 2450

Commit message: Fixed footprints for tecminal blocks
Parts:
- added R12, R13, R14, R15: 10K, Resistors_SMD:R_0805_HandSoldering, symbol R
- P6: footprint Socket_Strips:Socket_Strip_Straight_1x02 -> Local:TERM_BLOCK_2
- P7: footprint Socket_Strips:Socket_Strip_Straight_1x08 -> Local:TERM_BLOCK_8
Connections:
- net GND: now also R12.1, R13.1, R14.1, R15.1
- net TRIGGER1: now also R12.2
- net TRIGGER2: now also R13.2
- net TRIGGER3: now also R14.2
- net TRIGGER4: now also R15.2
Changed lines of the file:
@@
 $Descr A4 11693 8268
 encoding utf-8
-Sheet 4 5
+Sheet 3 5
 Title ""
 Date "6 dec 2014"
@@
 Text Label 2000 3300 2    60   ~ 0
 V_PYRO
-Wire Wire Line
-	1300 3500 1400 3500
-Wire Wire Line
-	1400 3500 1400 3600
-Wire Wire Line
-	1400 2500 1750 2500
-Wire Wire Line
-	1400 1750 1400 2000
-Wire Wire Line
-	1400 2000 2050 2000
-Wire Wire Line
-	2050 2000 2050 2250
-Wire Wire Line
-	1400 2850 1450 2850
-Connection ~ 2050 2850
-Wire Wire Line
-	700  1750 700  2500
-Wire Wire Line
-	700  2500 900  2500
-Wire Wire Line
-	1200 2650 1200 2950
-Wire Wire Line
-	1400 2100 1400 2850
-Wire Wire Line
-	1950 2850 2050 2850
-Wire Wire Line
-	1200 2950 9000 2950
-Connection ~ 2050 2950
-Wire Wire Line
-	1200 2100 2650 2100
-Wire Wire Line
-	1200 2100 1200 2250
-Wire Wire Line
-	2650 2100 2650 3550
-Wire Wire Line
-	1300 3300 3350 3300
-Wire Wire Line
-	2750 3300 2750 3550
-Wire Wire Line
-	2950 3300 2950 3550
-Connection ~ 2750 3300
-Wire Wire Line
-	3150 3300 3150 3550
-Connection ~ 2950 3300
-Wire Wire Line
-	3350 3300 3350 3550
-Connection ~ 3150 3300
-Connection ~ 1400 2500
-Connection ~ 1400 2100
-Wire Wire Line
-	1300 2250 1300 2100
-Connection ~ 1300 2100
-Wire Wire Line
-	3850 2500 4200 2500
-Wire Wire Line
-	3850 1750 3850 2000
-Wire Wire Line
-	3850 2000 4500 2000
-Wire Wire Line
-	4500 2000 4500 2250
-Wire Wire Line
-	4500 2650 4500 3000
-Wire Wire Line
-	3850 2850 3900 2850
-Connection ~ 4500 2850
-Wire Wire Line
-	3150 2500 3350 2500
-Wire Wire Line
-	3650 2950 3650 2650
-Wire Wire Line
-	3850 2100 3850 2850
-Wire Wire Line
-	4400 2850 4500 2850
-Connection ~ 4500 2950
-Wire Wire Line
-	3650 2100 5100 2100
-Wire Wire Line
-	3650 2100 3650 2250
-Connection ~ 3850 2500
-Connection ~ 3850 2100
-Wire Wire Line
-	3750 2250 3750 2100
-Connection ~ 3750 2100
-Wire Wire Line
-	5100 2100 5100 3150
-Wire Wire Line
-	5100 3150 2850 3150
-Wire Wire Line
-	2850 3150 2850 3550
-Wire Wire Line
-	6100 2500 6450 2500
-Wire Wire Line
-	6100 1750 6100 2000
-Wire Wire Line
-	6100 2000 6750 2000
-Wire Wire Line
-	6750 2000 6750 2250
-Wire Wire Line
-	6100 2850 6150 2850
-Connection ~ 6750 2850
-Wire Wire Line
-	5400 1750 5400 2500
-Wire Wire Line
-	5400 2500 5600 2500
-Wire Wire Line
-	5900 2950 5900 2650
-Wire Wire Line
-	6100 2100 6100 2850
-Wire Wire Line
-	6650 2850 6750 2850
-Connection ~ 6750 2950
-Wire Wire Line
-	5900 2100 7350 2100
-Wire Wire Line
-	5900 2100 5900 2250
-Connection ~ 6100 2500
-Connection ~ 6100 2100
-Wire Wire Line
-	6000 2250 6000 2100
-Connection ~ 6000 2100
-Wire Wire Line
-	3050 3550 3050 3200
-Wire Wire Line
-	3050 3200 7350 3200
-Wire Wire Line
-	8350 2500 8700 2500
-Wire Wire Line
-	8350 1750 8350 2000
-Wire Wire Line
-	8350 2000 9000 2000
-Wire Wire Line
-	9000 2000 9000 2250
-Wire Wire Line
-	8350 2850 8400 2850
-Connection ~ 9000 2850
-Wire Wire Line
-	7650 1750 7650 2500
-Wire Wire Line
-	7650 2500 7850 2500
-Wire Wire Line
-	8150 2950 8150 2650
-Wire Wire Line
-	8350 2100 8350 2850
-Wire Wire Line
-	8900 2850 9000 2850
-Connection ~ 9000 2950
-Wire Wire Line
-	8150 2100 9600 2100
-Wire Wire Line
-	8150 2100 8150 2250
-Connection ~ 8350 2500
-Connection ~ 8350 2100
-Wire Wire Line
-	8250 2250 8250 2100
-Connection ~ 8250 2100
-Wire Wire Line
-	7350 3200 7350 2100
-Wire Wire Line
-	3250 3550 3250 3350
-Wire Wire Line
-	3250 3350 9600 3350
-Wire Wire Line
-	9600 3350 9600 2100
-Wire Wire Line
-	2050 2950 2050 2650
-Connection ~ 3650 2950
-Wire Wire Line
-	6750 2950 6750 2650
-Connection ~ 5900 2950
-Connection ~ 8150 2950
-Wire Wire Line
-	9000 2950 9000 2650
 $Comp
 L TERM_BLOCK_2.54MM_2POS P6
@@
 F 0 "P6" V 900 3400 40  0000 C CNN
 F 1 "TERM_BLOCK_2.54MM_2POS" V 1000 3400 40  0000 C CNN
-F 2 "Socket_Strips:Socket_Strip_Straight_1x02" H 950 3400 60  0001 C CNN
+F 2 "Local:TERM_BLOCK_2" H 950 3400 60  0001 C CNN
 F 3 "" H 950 3400 60  0000 C CNN
 	1    950  3400
@@
 F 0 "P7" V 2950 3900 60  0000 C CNN
 F 1 "TERM_BLOCK_2.54MM_8POS" V 3050 3900 60  0000 C CNN
-F 2 "Socket_Strips:Socket_Strip_Straight_1x08" H 3000 3900 60  0001 C CNN
+F 2 "Local:TERM_BLOCK_8" H 3000 3900 60  0001 C CNN
 F 3 "" H 3000 3900 60  0000 C CNN
 	1    3000 3900
@@
 	1    0    0    -1
 $EndComp
+$Comp
+L GND #PWR024
+U 1 1 550499F5
+P 950 850
+F 0 "#PWR024" H 950 850 30  0001 C CNN
+F 1 "GND" H 950 780 30  0001 C CNN
+F 2 "" H 950 850 60  0000 C CNN
+F 3 "" H 950 850 60  0000 C CNN
+	1    950  850
+	-1   0    0    1
+$EndComp
+$Comp
+L R R12
+U 1 1 55049B7A
+P 950 1400
+F 0 "R12" V 1030 1400 40  0000 C CNN
+F 1 "10K" V 957 1401 40  0000 C CNN
+F 2 "Resistors_SMD:R_0805_HandSoldering" V 880 1400 30  0001 C CNN
+F 3 "~" H 950 1400 30  0000 C CNN
+	1    950  1400
+	1    0    0    -1
+$EndComp
+$Comp
+L R R13
+U 1 1 55049C07
+P 3400 1400
+F 0 "R13" V 3480 1400 40  0000 C CNN
+F 1 "10K" V 3407 1401 40  0000 C CNN
+F 2 "Resistors_SMD:R_0805_HandSoldering" V 3330 1400 30  0001 C CNN
+F 3 "~" H 3400 1400 30  0000 C CNN
+	1    3400 1400
+	1    0    0    -1
+$EndComp
+$Comp
+L R R14
+U 1 1 55049C95
+P 5650 1400
+F 0 "R14" V 5730 1400 40  0000 C CNN
+F 1 "10K" V 5657 1401 40  0000 C CNN
+F 2 "Resistors_SMD:R_0805_HandSoldering" V 5580 1400 30  0001 C CNN
+F 3 "~" H 5650 1400 30  0000 C CNN
+	1    5650 1400
+	1    0    0    -1
+$EndComp
+$Comp
+L R R15
+U 1 1 55049DC7
+P 7900 1400
+F 0 "R15" V 7980 1400 40  0000 C CNN
+F 1 "10K" V 7907 1401 40  0000 C CNN
+F 2 "Resistors_SMD:R_0805_HandSoldering" V 7830 1400 30  0001 C CNN
+F 3 "~" H 7900 1400 30  0000 C CNN
+	1    7900 1400
+	1    0    0    -1
+$EndComp
+Wire Wire Line
+	1300 3500 1400 3500
+Wire Wire Line
+	1400 3500 1400 3600
+Wire Wire Line
+	1400 2500 1750 2500
+Wire Wire Line
+	1400 1750 1400 2000
+Wire Wire Line
+	1400 2000 2050 2000
+Wire Wire Line
+	2050 2000 2050 2250
+Wire Wire Line
+	1400 2850 1450 2850
+Connection ~ 2050 2850
+Wire Wire Line
+	700  1750 700  2500
+Wire Wire Line
+	700  2500 900  2500
+Wire Wire Line
+	1200 2650 1200 2950
+Wire Wire Line
+	1400 2100 1400 2850
+Wire Wire Line
+	1950 2850 2050 2850
+Wire Wire Line
+	1200 2950 9000 2950
+Connection ~ 2050 2950
+Wire Wire Line
+	1200 2100 2650 2100
+Wire Wire Line
+	1200 2100 1200 2250
+Wire Wire Line
+	2650 2100 2650 3550
+Wire Wire Line
+	1300 3300 3350 3300
+Wire Wire Line
+	2750 3300 2750 3550
+Wire Wire Line
+	2950 3300 2950 3550
+Connection ~ 2750 3300
+Wire Wire Line
+	3150 3300 3150 3550
+Connection ~ 2950 3300
+Wire Wire Line
+	3350 3300 3350 3550
+Connection ~ 3150 3300
+Connection ~ 1400 2500
+Connection ~ 1400 2100
+Wire Wire Line
+	1300 2250 1300 2100
+Connection ~ 1300 2100
+Wire Wire Line
+	3850 2500 4200 2500
+Wire Wire Line
+	3850 1750 3850 2000
+Wire Wire Line
+	3850 2000 4500 2000
+Wire Wire Line
+	4500 2000 4500 2250
+Wire Wire Line
+	4500 2650 4500 3000
+Wire Wire Line
+	3850 2850 3900 2850
+Connection ~ 4500 2850
+Wire Wire Line
+	3150 2500 3350 2500
+Wire Wire Line
+	3650 2950 3650 2650
+Wire Wire Line
+	3850 2100 3850 2850
+Wire Wire Line
+	4400 2850 4500 2850
+Connection ~ 4500 2950
+Wire Wire Line
+	3650 2100 5100 2100
+Wire Wire Line
+	3650 2100 3650 2250
+Connection ~ 3850 2500
+Connection ~ 3850 2100
+Wire Wire Line
+	3750 2250 3750 2100
+Connection ~ 3750 2100
+Wire Wire Line
+	5100 2100 5100 3150
+Wire Wire Line
+	5100 3150 2850 3150
+Wire Wire Line
+	2850 3150 2850 3550
+Wire Wire Line
+	6100 2500 6450 2500
+Wire Wire Line
+	6100 1750 6100 2000
+Wire Wire Line
+	6100 2000 6750 2000
+Wire Wire Line
+	6750 2000 6750 2250
+Wire Wire Line
+	6100 2850 6150 2850
+Connection ~ 6750 2850
+Wire Wire Line
+	5400 1750 5400 2500
+Wire Wire Line
+	5400 2500 5600 2500
+Wire Wire Line
+	5900 2950 5900 2650
+Wire Wire Line
+	6100 2100 6100 2850
+Wire Wire Line
+	6650 2850 6750 2850
+Connection ~ 6750 2950
+Wire Wire Line
+	5900 2100 7350 2100
+Wire Wire Line
+	5900 2100 5900 2250
+Connection ~ 6100 2500
+Connection ~ 6100 2100
+Wire Wire Line
+	6000 2250 6000 2100
+Connection ~ 6000 2100
+Wire Wire Line
+	3050 3550 3050 3200
+Wire Wire Line
+	3050 3200 7350 3200
+Wire Wire Line
+	8350 2500 8700 2500
+Wire Wire Line
+	8350 1750 8350 2000
+Wire Wire Line
+	8350 2000 9000 2000
+Wire Wire Line
+	9000 2000 9000 2250
+Wire Wire Line
+	8350 2850 8400 2850
+Connection ~ 9000 2850
+Wire Wire Line
+	7650 1750 7650 2500
+Wire Wire Line
+	7650 2500 7850 2500
+Wire Wire Line
+	8150 2950 8150 2650
+Wire Wire Line
+	8350 2100 8350 2850
+Wire Wire Line
+	8900 2850 9000 2850
+Connection ~ 9000 2950
+Wire Wire Line
+	8150 2100 9600 2100
+Wire Wire Line
+	8150 2100 8150 2250
+Connection ~ 8350 2500
+Connection ~ 8350 2100
+Wire Wire Line
+	8250 2250 8250 2100
+Connection ~ 8250 2100
+Wire Wire Line
+	7350 3200 7350 2100
+Wire Wire Line
+	3250 3550 3250 3350
+Wire Wire Line
+	3250 3350 9600 3350
+Wire Wire Line
+	9600 3350 9600 2100
+Wire Wire Line
+	2050 2950 2050 2650
+Connection ~ 3650 2950
+Wire Wire Line
+	6750 2950 6750 2650
+Connection ~ 5900 2950
+Connection ~ 8150 2950
+Wire Wire Line
+	9000 2950 9000 2650
 Wire Wire Line
 	3150 1750 3150 2500
+Wire Wire Line
+	7900 1650 7900 1950
+Wire Wire Line
+	7900 1950 7650 1950
+Connection ~ 7650 1950
+Wire Wire Line
+	5650 1650 5650 1850
+Wire Wire Line
+	5650 1850 5400 1850
+Connection ~ 5400 1850
+Wire Wire Line
+	3400 1650 3400 1850
+Wire Wire Line
+	3400 1850 3150 1850
+Connection ~ 3150 1850
+Wire Wire Line
+	950  1650 950  1850
+Wire Wire Line
+	950  1850 700  1850
+Connection ~ 700  1850
+Wire Wire Line
+	950  1150 950  850
+Wire Wire Line
+	950  1050 7900 1050
+Wire Wire Line
+	3400 1050 3400 1150
+Connection ~ 950  1050
+Wire Wire Line
+	5650 1050 5650 1150
+Connection ~ 3400 1050
+Wire Wire Line
+	7900 1050 7900 1150
+Connection ~ 5650 1050
 $EndSCHEMATC
