File: Hardware/mcu.sch (KiCad schematic (older format))
At the start: 10 parts, among them SW3 SW_PUSH, U1 STM32F411RE_LQFP64

Commit message: Began routing
Changed lines of the file:
@@
 $EndDescr
 $Comp
-L 3V3 #PWR021
+L 3V3 #PWR024
 U 1 1 542CDA8F
 P 3800 3600
-F 0 "#PWR021" H 3800 3700 40  0001 C CNN
+F 0 "#PWR024" H 3800 3700 40  0001 C CNN
 F 1 "3V3" H 3800 3725 40  0000 C CNN
 F 2 "" H 3800 3600 60  0000 C CNN
@@
 $EndComp
 $Comp
-L GND #PWR022
+L GND #PWR025
 U 1 1 542CDA9E
 P 3850 3850
-F 0 "#PWR022" H 3850 3850 30  0001 C CNN
+F 0 "#PWR025" H 3850 3850 30  0001 C CNN
 F 1 "GND" H 3850 3780 30  0001 C CNN
 F 2 "" H 3850 3850 60  0000 C CNN
@@
 $EndComp
 $Comp
-L 3V3 #PWR023
+L 3V3 #PWR026
 U 1 1 542CDAB1
 P 3800 4800
-F 0 "#PWR023" H 3800 4900 40  0001 C CNN
+F 0 "#PWR026" H 3800 4900 40  0001 C CNN
 F 1 "3V3" H 3800 4925 40  0000 C CNN
 F 2 "" H 3800 4800 60  0000 C CNN
@@
 $EndComp
 $Comp
-L 3V3 #PWR024
+L 3V3 #PWR027
 U 1 1 542CDAB7
 P 7450 4850
-F 0 "#PWR024" H 7450 4950 40  0001 C CNN
+F 0 "#PWR027" H 7450 4950 40  0001 C CNN
 F 1 "3V3" H 7450 4975 40  0000 C CNN
 F 2 "" H 7450 4850 60  0000 C CNN
@@
 $EndComp
 $Comp
-L 3V3 #PWR025
+L 3V3 #PWR028
 U 1 1 542CDC4D
 P 7500 3350
-F 0 "#PWR025" H 7500 3450 40  0001 C CNN
+F 0 "#PWR028" H 7500 3450 40  0001 C CNN
 F 1 "3V3" H 7500 3475 40  0000 C CNN
 F 2 "" H 7500 3350 60  0000 C CNN
@@
 $EndComp
 $Comp
-L GND #PWR026
+L GND #PWR029
 U 1 1 5430D873
 P 6150 1450
-F 0 "#PWR026" H 6150 1450 30  0001 C CNN
+F 0 "#PWR029" H 6150 1450 30  0001 C CNN
 F 1 "GND" H 6150 1380 30  0001 C CNN
 F 2 "" H 6150 1450 60  0000 C CNN
@@
 $EndComp
 $Comp
-L 3V3 #PWR027
+L 3V3 #PWR030
 U 1 1 5430DC01
 P 7600 4350
-F 0 "#PWR027" H 7600 4450 40  0001 C CNN
+F 0 "#PWR030" H 7600 4450 40  0001 C CNN
 F 1 "3V3" H 7600 4475 40  0000 C CNN
 F 2 "" H 7600 4350 60  0000 C CNN
@@
 $EndComp
 $Comp
-L GND #PWR028
+L GND #PWR031
 U 1 1 5430DC07
 P 9000 4500
-F 0 "#PWR028" H 9000 4500 30  0001 C CNN
+F 0 "#PWR031" H 9000 4500 30  0001 C CNN
 F 1 "GND" H 9000 4430 30  0001 C CNN
 F 2 "" H 9000 4500 60  0000 C CNN
@@
 $EndComp
 $Comp
-L 3V3 #PWR029
+L 3V3 #PWR032
 U 1 1 5430E0CC
 P 5300 5450
-F 0 "#PWR029" H 5300 5550 40  0001 C CNN
+F 0 "#PWR032" H 5300 5550 40  0001 C CNN
 F 1 "3V3" H 5300 5575 40  0000 C CNN
 F 2 "" H 5300 5450 60  0000 C CNN
@@
 $EndComp
 $Comp
-L GND #PWR030
+L GND #PWR033
 U 1 1 5430E365
 P 5300 6050
-F 0 "#PWR030" H 5300 6050 30  0001 C CNN
+F 0 "#PWR033" H 5300 6050 30  0001 C CNN
 F 1 "GND" H 5300 5980 30  0001 C CNN
 F 2 "" H 5300 6050 60  0000 C CNN
@@
 $EndComp
 $Comp
-L GND #PWR031
+L GND #PWR034
 U 1 1 5430E5BA
 P 3550 4650
-F 0 "#PWR031" H 3550 4650 30  0001 C CNN
+F 0 "#PWR034" H 3550 4650 30  0001 C CNN
 F 1 "GND" H 3550 4580 30  0001 C CNN
 F 2 "" H 3550 4650 60  0000 C CNN
@@
 USART_RX
 $Comp
-L 3V3 #PWR032
+L 3V3 #PWR035
 U 1 1 5430E17B
 P 4050 1800
-F 0 "#PWR032" H 4050 1900 40  0001 C CNN
+F 0 "#PWR035" H 4050 1900 40  0001 C CNN
 F 1 "3V3" H 4050 1925 40  0000 C CNN
 F 2 "" H 4050 1800 60  0000 C CNN
@@
 	4150 4900 4150 5300
 $Comp
-L GND #PWR033
+L GND #PWR036
 U 1 1 54449600
 P 4150 5300
-F 0 "#PWR033" H 4150 5300 30  0001 C CNN
+F 0 "#PWR036" H 4150 5300 30  0001 C CNN
 F 1 "GND" H 4150 5230 30  0001 C CNN
 F 2 "" H 4150 5300 60  0000 C CNN
@@
 	7350 4900 7350 5100
 $Comp
-L GND #PWR034
+L GND #PWR037
 U 1 1 5444A762
 P 7350 3600
-F 0 "#PWR034" H 7350 3600 30  0001 C CNN
+F 0 "#PWR037" H 7350 3600 30  0001 C CNN
 F 1 "GND" H 7350 3530 30  0001 C CNN
 F 2 "" H 7350 3600 60  0000 C CNN
@@
 	7350 3300 7350 3600
 $Comp
-L GND #PWR035
+L GND #PWR038
 U 1 1 54449656
 P 7350 5100
-F 0 "#PWR035" H 7350 5100 30  0001 C CNN
+F 0 "#PWR038" H 7350 5100 30  0001 C CNN
 F 1 "GND" H 7350 5030 30  0001 C CNN
 F 2 "" H 7350 5100 60  0000 C CNN
@@
 Text HLabel 8800 5250 2    60   Input ~ 0
 SYS_SDA
+Text HLabel 4150 3100 0    60   Input ~ 0
+VDDA
 Text HLabel 4150 3000 0    60   Input ~ 0
-VDDA
-Text HLabel 4150 3100 0    60   Input ~ 0
 VSSA
 $EndSCHEMATC

Commit message: Ready to begin laying out and routing
Parts:
- SW3: footprint Discret:SW_PUSH_SMALL -> Local:SW_SMD_MICRO
Changed lines of the file:
@@
 F 0 "SW3" H 5900 1210 50  0000 C CNN
 F 1 "SW_PUSH" H 5750 1020 50  0000 C CNN
-F 2 "Discret:SW_PUSH_SMALL" H 5750 1100 60  0001 C CNN
+F 2 "Local:SW_SMD_MICRO" H 5750 1100 60  0001 C CNN
 F 3 "~" H 5750 1100 60  0000 C CNN
 	1    5750 1100
